File: Hardware/Milli_Matrix_v2.sch (EAGLE design)
At the start: 40 parts, among them U1 ATMEGA32U4QFN2, U2 MCP73831, U3 MIC5219-3.3, Y1 8MHz

Commit message: PCB Cleanup + back solder pads for mounting
Tweaked some of the component placements

Put some rectangles on the back of the board in hopes of soldering
safety pins to them.
Parts:
- JP6, JP7: value FIDUCIAL1.5X3 -> FIDUCIAL1X2; device SparkFun:FIDUCIAL1.5X3 -> SparkFun:FIDUCIAL1X2
Changed lines of the file:
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@@
 <part name="GND9" library="SparkFun" deviceset="GND" device=""/>
 <part name="P+9" library="SparkFun" deviceset="3.3V" device="" value="VCC"/>
-<part name="JP6" library="SparkFun" deviceset="FIDUCIAL" device="1.5X3"/>
-<part name="JP7" library="SparkFun" deviceset="FIDUCIAL" device="1.5X3"/>
+<part name="JP6" library="SparkFun" deviceset="FIDUCIAL" device="1X2"/>
+<part name="JP7" library="SparkFun" deviceset="FIDUCIAL" device="1X2"/>
 <part name="FRAME1" library="frames" deviceset="A3L-LOC" device=""/>
 </parts>
